Commit message: added lidar

File: models/robot_manipulator/robot_manipulator.urdf (robot description, URDF)
Before this commit: robot robot_manipulator, 6 links, 5 joints
Links:
- added link lidar, mass 0.25; collision cylinder length=0.03 radius=0.04; visual cylinder length=0.03 radius=0.04
- added link lidar_mount_link, mass 0.001
Joints:
- added joint lidar_joint: type fixed, parent lidar_mount_link, child lidar, origin xyz=0 0 0.02 rpy=0 0 0
- added joint lidar_mount_joint: type fixed, parent base_link, child lidar_mount_link, origin xyz=0.2 0 0.075 rpy=0 0 0

File: urdf/robot_manipulator.urdf.xacro (robot description, xacro)
@@ -3,4 +3,5 @@
 	<xacro:include filename="$(find robot_manipulator)/urdf/wheels.xacro"/>
 	<xacro:include filename="$(find robot_manipulator)/urdf/caster_wheels.xacro"/>
+	<xacro:include filename="$(find robot_manipulator)/urdf/lidar.xacro"/>
 	<link name="base_footprint" />
 	<joint name="base_joint" type="fixed">
@@ -70,3 +71,7 @@
 		</plugin>
 	</gazebo>
+	<!-- Sensors -->
+	<xacro:lidar_sensor name="lidar" parent="base_link" >
+		<origin xyz="0.2 0 0.075" rpy="0 0 0"/>
+	</xacro:lidar_sensor>
 </robot>
